Commit message: custom modi -2

File: src/piper_description/urdf/piper_description_d405.xacro (robot description, xacro)
@@ -3,5 +3,5 @@
   name="piper"
   xmlns:xacro="http://ros.org/wiki/xacro">
-    <xacro:include filename="$(find realsense_custom_description)/urdf/test_d435i_camera.urdf.xacro"/>
+    <xacro:include filename="$(find realsense_custom_description)/urdf/test_d405_camera.urdf.xacro"/>
 <!-- world -->
   <link name="world"/>
@@ -11,8 +11,10 @@
   </joint>
 <!-- 相機與第六軸連接 -->
-<joint name="d435_joint" type="fixed">
-    <origin xyz="-0.080 0.0669 -0.2959" rpy="-0.3358 0.00566 -1.6549"/>
+<joint name="d405_joint" type="fixed">
+    <!--  <origin xyz="-0.064868 0.014226 0.029185" rpy="-0.283249 0.012335 -1.670768"/>
+    <origin xyz="-0.06092 0.00551 0.030946" rpy="-0.29119 0.016918 -1.6641"/>-->
+    <origin xyz="-0.055 0.0144 0.0082" rpy="-0.253 0.0632 -1.635"/>
     <parent link="link6"/>
-    <child link="d435_base_link"/>
+    <child link="d405_base_link"/>
 </joint>
 <!-- arm -->

File: src/realsense_custom_description/urdf/test_d435i_camera.urdf.xacro (robot description, xacro)
@@ -3,7 +3,7 @@
   <xacro:arg name="use_nominal_extrinsics" default="false" />
   <xacro:include filename="$(find realsense2_description)/urdf/_d435i.urdf.xacro"/>
-  <link name="base_link" />
-  <xacro:sensor_d435i parent="base_link" use_nominal_extrinsics="$(arg use_nominal_extrinsics)">
-    <origin xyz="0 0 0" rpy="0 0 0"/>
+  <link name="d435_base_link" />
+  <xacro:sensor_d435i parent="d435_base_link" use_nominal_extrinsics="$(arg use_nominal_extrinsics)">
+    <origin xyz="0 0 0" rpy="0 -1.57 1.57"/>
   </xacro:sensor_d435i>
 </robot>

Commit message: curobo_version

File: src/piper_description/urdf/piper_description_d405.xacro (robot description, xacro)
@@ -12,7 +12,7 @@
 <!-- 相機與第六軸連接 -->
 <joint name="d405_joint" type="fixed">
-    <!--  <origin xyz="-0.064868 0.014226 0.029185" rpy="-0.283249 0.012335 -1.670768"/>
-    <origin xyz="-0.06092 0.00551 0.030946" rpy="-0.29119 0.016918 -1.6641"/>-->
-    <origin xyz="-0.055 0.0144 0.0082" rpy="-0.253 0.0632 -1.635"/>
+      <!--<origin xyz="-0.064868 0.014226 0.029185" rpy="-0.283249 0.012335 -1.670768"/> -->
+   <origin xyz="-0.06092 0.00551 0.030946" rpy="-0.29119 0.016918 -1.6641"/>
+     <!--<origin xyz="-0.055 0.0144 0.0082" rpy="-0.253 0.0632 -1.635"/>-->
     <parent link="link6"/>
     <child link="d405_base_link"/>
@@ -95,5 +95,5 @@
     <limit
       lower="-2.618"
-      upper="2.168"
+      upper="2.618"
       effort="100"
       velocity="5" />
@@ -414,5 +414,5 @@
       <origin
         xyz="0 0 0"
-        rpy="0 0 0" />
+        rpy="1.5708 0 0" />
       <geometry>
         <mesh
@@ -440,5 +440,5 @@
     <origin
       xyz="0 0 0.1358"
-      rpy="1.5708 0 0" />
+      rpy="0 0 0" />
     <parent
       link="gripper_base" />
@@ -446,8 +446,8 @@
       link="link7" />
     <axis
-      xyz="0 0 1" />
-    <limit
-      lower="0"
-      upper="0.09"
+      xyz="0 1 0" />
+    <limit
+      lower="-0.09"
+      upper="0"
       effort="10"
       velocity="1" />

File: src/piper_description/urdf/piper_description_d435.xacro (robot description, xacro)
@@ -12,5 +12,5 @@
 <!-- 相機與第六軸連接 -->
 <joint name="d435_joint" type="fixed">
-    <origin xyz="-0.080 0.0669 -0.2959" rpy="-0.3358 0.00566 -1.6549"/>
+    <origin xyz="-0.080 0.0669 -0.0473" rpy="-0.3448 0.0184 -1.536"/>
     <parent link="link6"/>
     <child link="d435_base_link"/>
