Commit message: Add triple arm version

File: src/Dual-arm-robot/scout_description/urdf/combined_robot_doublearm_nocar.urdf (robot description, URDF)
Before this commit: robot combined_robot, 42 links, 41 joints
Links:
- removed link Livox_mid_360
- removed link combined_base
- removed link front_left_wheel_link
- removed link front_mount
- removed link front_right_wheel_link
- removed link inertial_link
- removed link link3_1_v1_1
- removed link link5_1_v1_1
- removed link link_1_1
- removed link link_2_1
- removed link link_4_1_1_v1_1
- removed link rear_left_wheel_link
- removed link rear_mount
- removed link rear_right_wheel_link
- removed link zyx_R_1_base_link
- added link arm1_gripper_point
- added link arm2_gripper_point
- added link link1_v1_1, mass 0.4200298104778203; collision mesh filename=file:///home/ros2/ros2_workspace/official_piper_ws/install/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 scale=0.001 0.001 0.001; visual mesh filename=file:///home/ros2/ros2_workspace/official_piper_ws/install/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 scale=0.001 0.001 0.001
- added link link2_3_v4_1, mass 1.8966297326812738; collision mesh filename=file:///home/ros2/ros2_workspace/official_piper_ws/install/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 scale=0.001 0.001 0.001; visual mesh filename=file:///home/ros2/ros2_workspace/official_piper_ws/install/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 scale=0.001 0.001 0.001
- added link link4_v3_1, mass 0.9123222504571403; collision mesh filename=file:///home/ros2/ros2_workspace/official_piper_ws/install/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 scale=0.001 0.001 0.001; visual mesh filename=file:///home/ros2/ros2_workspace/official_piper_ws/install/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 scale=0.001 0.001 0.001
- added link link5_v3_1, mass 1.0415582650622635; collision mesh filename=file:///home/ros2/ros2_workspace/official_piper_ws/install/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 scale=0.001 0.001 0.001; visual mesh filename=file:///home/ros2/ros2_workspace/official_piper_ws/install/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 scale=0.001 0.001 0.001
- added link link6_v3_1, mass 0.792974216910335; collision mesh filename=file:///home/ros2/ros2_workspace/official_piper_ws/install/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 scale=0.001 0.001 0.001; visual mesh filename=file:///home/ros2/ros2_workspace/official_piper_ws/install/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 scale=0.001 0.001 0.001
- link base_link: mass None -> 37.77937726543091; geometry collision mesh filename=file:///home/ros2/ros2_workspace/official_piper_ws/install/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 scale=0.001 0.001 0.001; visual mesh filename=file:///home/ros2/ros2_workspace/official_piper_ws/install/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 scale=0.001 0.001 0.001
Joints:
- removed joint G
- removed joint R
- removed joint X
- removed joint Y
- removed joint Z
- removed joint front_left_wheel
- removed joint front_mount_joint
- removed joint front_right_wheel
- removed joint inertial_joint
- removed joint lidar_joint
- removed joint rear_left_wheel
- removed joint rear_mount_joint
- removed joint rear_right_wheel
- removed joint scout_v2_base_joint
- removed joint zyx_R_1_base_joint
- added joint Revolute 1: type revolute, parent base_link, child link1_v1_1, origin xyz=0.0 0.0 0.0815 rpy=0 0 -1.57, axis -0.0 0.0 1.0, limit lower=-2.96706 upper=3.054326 effort=100 velocity=100
- added joint Revolute 2: type revolute, parent link1_v1_1, child link2_3_v4_1, origin xyz=-0.011639 0.034477 0.0285 rpy=0 0 0, axis 1.0 0.0 0.0, limit lower=-1.745329 upper=1.308997 effort=100 velocity=100
- added joint Revolute 3: type revolute, parent link2_3_v4_1, child link4_v3_1, origin xyz=0.03565 0.0 0.168 rpy=0 0 0, axis 1.0 -0.0 0.0, limit lower=-1.570796 upper=1.396263 effort=100 velocity=100
- added joint Revolute 4: type revolute, parent link4_v3_1, child link5_v3_1, origin xyz=-0.013162 0.001043 0.062467 rpy=0 0 0, axis -0.0 1.0 0.0, limit lower=-3.141593 upper=3.141593 effort=100 velocity=100
- added joint Revolute 5: type revolute, parent link5_v3_1, child link6_v3_1, origin xyz=0.0223 0.11 0.0 rpy=0 0 0, axis 1.0 0.0 0.0, limit lower=-1.745329 upper=1.919862 effort=100 velocity=100
- added joint arm1_gripper_points: type fixed, parent arm1_link6, child arm1_gripper_point, origin xyz=-0.0 0.0 0.11 rpy=-0.0 0.0 -3.14
- added joint arm2_gripper_points: type fixed, parent arm2_link6, child arm2_gripper_point, origin xyz=-0.0 0.0 0.11 rpy=-0.0 0.0 -3.14
- joint arm1_fixed_base_joint: origin xyz=0.0 -0.20 0.05 rpy=0 0 0 -> xyz=0.0075 0.21 -0.075 rpy=3.14 0 0; parent link3_1_v1_1 -> base_link
- joint arm2_fixed_base_joint: origin xyz=0.0 0.20 0.05 rpy=0 0 0 -> xyz=0.0075 -0.21 -0.075 rpy=3.14 0 0; parent link3_1_v1_1 -> base_link
- joint cam1_d405_joint: origin xyz=-0.06092 0.00551 0.030946 rpy=-0.29119 0.016918 -1.6641 -> xyz=-0.10152 0.00327 0.030479 rpy=0.29119 -0.020223 1.433
- joint cam2_d405_joint: origin xyz=-0.06092 0.00551 0.030946 rpy=-0.29119 0.016918 -1.6641 -> xyz=-0.10152 0.00327 0.030479 rpy=0.29119 -0.020223 1.57

File: src/Dual-arm-robot/scout_description/urdf/combined_robot_doublearm_nocar.xacro (robot description, xacro)
@@ -6,9 +6,12 @@
   <!-- <xacro:include filename="$(find piper_description)/urdf/piper_description.xacro"/>-->
     <!-- 引入 piper_arm_macro.xacro-->
+    <xacro:include filename="$(find Dual_piper_ROS2_description)/urdf/materials.xacro" />
+<xacro:include filename="$(find Dual_piper_ROS2_description)/urdf/Dual_piper_ROS2.trans" />
+<xacro:include filename="$(find Dual_piper_ROS2_description)/urdf/Dual_piper_ROS2.gazebo" />
       <xacro:include filename="$(find realsense2_description)/urdf/_materials.urdf.xacro" />
 <xacro:include filename="$(find piper_description)/urdf/piper_description_d405_marco.xacro"/>
   <!-- 引入相機的Xacro文件 -->
 <xacro:include filename="$(find realsense_custom_description)/urdf/piper_double_d405_camera.urdf.xacro"/>
-  <!-- 定義統一的父連接點 -->
+  <!-- 定義統一的父連接點
   <link name="base_link">
     <inertial>
@@ -17,10 +20,39 @@
     </inertial>
   </link>
-<!-- 在 link3_1_v1_1 左邊掛載第一支手臂 -->
+-->
+<link name="base_link">
+  <inertial>
+    <origin xyz="-0.0023454168511469727 -7.5124051764860745e-06 -0.20653047899548718" rpy="0 0 0"/>
+    <mass value="37.77937726543091"/>
+    <inertia ixx="2.333472" iyy="2.671087" izz="0.432453" ixy="-7e-06" iyz="0.006346" ixz="0.021116"/>
+  </inertial>
+  <visual>
+    <origin xyz="0 0 0" rpy="0 0 -1.57"/>
+    <geometry>
+      <!-- <mesh filename="file://$(find Dual_piper_ROS2_description)/meshes/base_link.stl" scale="0.001 0.001 0.001"/> -->
+      <mesh filename="file://$(find dummy_piper_ROS2_description)/meshes/base_link.stl" scale="0.001 0.001 0.001"/>
+    </geometry>
+    <material name="silver"/>
+  </visual>
+  <collision>
+    <origin xyz="0 0 0" rpy="0 0 -1.57"/>
+    <geometry>
+      <mesh filename="file://$(find Dual_piper_ROS2_description)/meshes/base_link.stl" scale="0.001 0.001 0.001"/>
+    </geometry>
+  </collision>
+</link>
+<!-- 在 link3_1_v1_1 左邊掛載第一支手臂
+<origin xyz="0.21 -0.0075 0.052" rpy="0 0 0"/>-->
   <xacro:piper_arm
     prefix="arm1"
     parent_link="base_link"
+    xyz="0.0075 0.21 -0.075"
+    rpy="3.14 0 0"/>
+    <!--
+  <xacro:piper_arm
+    prefix="arm1"
+    parent_link="base_link"
     xyz="0.0 -0.200 0.05"
-    rpy="3.14 0 0"/>
+    rpy="3.14 0 0"/>-->
     <!--rpy="0 0 0"/>-->
  <!-- 第1台相機：掛在 arm1link6
@@ -35,5 +67,10 @@
     roll="0.29119" pitch="-0.020223" yaw="1.433"
     use_nominal_extrinsics="false"/>
-  <!-- 在 link3_1_v1_1 右邊掛載第二支手臂  -->
+   <xacro:piper_arm
+    prefix="arm2"
+    parent_link="base_link"
+   xyz="0.0075 -0.21 -0.075"
+   rpy="3.14 0 0"/>
+  <!-- 在 link3_1_v1_1 右邊掛載第二支手臂
   <xacro:piper_arm
     prefix="arm2"
@@ -41,4 +78,5 @@
    xyz="0.0 0.200 0.05"
    rpy="3.14 0 0"/>
+   -->
     <!--  rpy="0 0 0"/> -->
     <!-- 第2台相機：掛在 arm2link6 -->
@@ -54,4 +92,163 @@
     roll="0.29119" pitch="-0.020223" yaw="1.57"
     use_nominal_extrinsics="false"/>
+    <link name="link1_v1_1">
+  <inertial>
+    <origin xyz="-0.005698056046029529 0.00648616381647002 0.012857188251092194" rpy="0 0 0"/>
+    <mass value="0.4200298104778203"/>
+    <inertia ixx="0.000188" iyy="0.000156" izz="0.000263" ixy="6.2e-05" iyz="-4.3e-05" ixz="2.7e-05"/>
+  </inertial>
+  <visual>
+    <origin xyz="0.0 0.0 -0.0815" rpy="0 0 0"/>
+    <geometry>
+      <mesh filename="file://$(find dummy_piper_ROS2_description)/meshes/link1_v1_1.stl" scale="0.001 0.001 0.001"/>
+    </geometry>
+    <material name="silver"/>
+  </visual>
+  <collision>
+    <origin xyz="0.0 0.0 -0.0815" rpy="0 0 0"/>
+    <geometry>
+      <mesh filename="file://$(find dummy_piper_ROS2_description)/meshes/link1_v1_1.stl" scale="0.001 0.001 0.001"/>
+    </geometry>
+  </collision>
+</link>
+<link name="link2_3_v4_1">
+  <inertial>
+    <origin xyz="0.01884442516054531 0.0019841485543513476 0.08366314329154632" rpy="0 0 0"/>
+    <mass value="1.8966297326812738"/>
+    <inertia ixx="0.00634" iyy="0.006744" izz="0.001194" ixy="-4e-06" iyz="6.4e-05" ixz="0.000771"/>
+  </inertial>
+  <visual>
+    <origin xyz="0.011639 -0.034477 -0.11" rpy="0 0 0"/>
+    <geometry>
+      <mesh filename="file://$(find dummy_piper_ROS2_description)/meshes/link2_3_v4_1.stl" scale="0.001 0.001 0.001"/>
+    </geometry>
+    <material name="silver"/>
+  </visual>
+  <collision>
+    <origin xyz="0.011639 -0.034477 -0.11" rpy="0 0 0"/>
+    <geometry>
+      <mesh filename="file://$(find dummy_piper_ROS2_description)/meshes/link2_3_v4_1.stl" scale="0.001 0.001 0.001"/>
+    </geometry>
+  </collision>
+</link>
+<link name="link4_v3_1">
+  <inertial>
+    <origin xyz="-0.010734927861478581 -0.02899910919329477 0.049078739095576474" rpy="0 0 0"/>
+    <mass value="0.9123222504571403"/>
+    <inertia ixx="0.00082" iyy="0.000695" izz="0.00053" ixy="-4.2e-05" iyz="0.000139" ixz="8.7e-05"/>
+  </inertial>
+  <visual>
+    <origin xyz="-0.024011 -0.034477 -0.278" rpy="0 0 0"/>
+    <geometry>
+      <mesh filename="file://$(find dummy_piper_ROS2_description)/meshes/link4_v3_1.stl" scale="0.001 0.001 0.001"/>
+    </geometry>
+    <material name="silver"/>
+  </visual>
+  <collision>
+    <origin xyz="-0.024011 -0.034477 -0.278" rpy="0 0 0"/>
+    <geometry>
+      <mesh filename="file://$(find dummy_piper_ROS2_description)/meshes/link4_v3_1.stl" scale="0.001 0.001 0.001"/>
+    </geometry>
+  </collision>
+</link>
+<link name="link5_v3_1">
+  <inertial>
+    <origin xyz="-0.0050623285902477895 0.05998132886165671 0.0006226400248250941" rpy="0 0 0"/>
+    <mass value="1.0415582650622635"/>
+    <inertia ixx="0.001817" iyy="0.000592" izz="0.002009" ixy="0.000108" iyz="-1.2e-05" ixz="8e-06"/>
+  </inertial>
+  <visual>
+    <origin xyz="-0.010849 -0.03552 -0.340467" rpy="0 0 0"/>
+    <geometry>
+      <mesh filename="file://$(find dummy_piper_ROS2_description)/meshes/link5_v3_1.stl" scale="0.001 0.001 0.001"/>
+    </geometry>
+    <material name="silver"/>
+  </visual>
+  <collision>
+    <origin xyz="-0.010849 -0.03552 -0.340467" rpy="0 0 0"/>
+    <geometry>
+      <mesh filename="file://$(find dummy_piper_ROS2_description)/meshes/link5_v3_1.stl" scale="0.001 0.001 0.001"/>
+    </geometry>
+  </collision>
+</link>
+<link name="link6_v3_1">
+  <inertial>
+    <origin xyz="-0.015134812773935424 0.07204733917419309 5.24783880485602e-05" rpy="0 0 0"/>
+    <mass value="0.792974216910335"/>
+    <inertia ixx="0.000883" iyy="0.000353" izz="0.000975" ixy="0.000146" iyz="1e-06" ixz="-0.0"/>
+  </inertial>
+  <visual>
+    <origin xyz="-0.033149 -0.14552 -0.340467" rpy="0 0 0"/>
+    <geometry>
+      <mesh filename="file://$(find dummy_piper_ROS2_description)/meshes/link6_v3_1.stl" scale="0.001 0.001 0.001"/>
+    </geometry>
+    <material name="silver"/>
+  </visual>
+  <collision>
+    <origin xyz="-0.033149 -0.14552 -0.340467" rpy="0 0 0"/>
+    <geometry>
+      <mesh filename="file://$(find dummy_piper_ROS2_description)/meshes/link6_v3_1.stl" scale="0.001 0.001 0.001"/>
+    </geometry>
+  </collision>
+</link>
+<link name="link7_v3_1">
+  <inertial>
+    <origin xyz="-0.015134812773935424 0.07204733917419309 5.24783880485602e-05" rpy="0 0 0"/>
+    <mass value="0.792974216910335"/>
+    <inertia ixx="0.000883" iyy="0.000353" izz="0.000975" ixy="0.000146" iyz="1e-06" ixz="-0.0"/>
+  </inertial>
+  <visual>
+    <origin xyz="-0.043149 -0.14552 -0.340467" rpy="0 0 0"/>
+    <geometry>
+      <!-- 使用簡單的盒子作為視覺參考 -->
+      <box size="0.01 0.01 0.01"/>
+    </geometry>
+    <material name="transparent">
+      <color rgba="0.0 0.0 0.0 0.0"/>  <!-- 完全透明 -->
+    </material>
+  </visual>
+</link>
+<joint name="dummy_joint1" type="revolute">
+  <origin xyz="0.0 0.0 0.0815" rpy="0 0 -1.57"/>
+  <parent link="base_link"/>
+  <child link="link1_v1_1"/>
+  <axis xyz="-0.0 0.0 1.0"/>
+  <limit upper="3.054326" lower="-2.96706" effort="100" velocity="100"/>
+</joint>
+<joint name="dummy_joint2" type="revolute">
+  <origin xyz="-0.011639 0.034477 0.0285" rpy="0 0 0"/>
+  <parent link="link1_v1_1"/>
+  <child link="link2_3_v4_1"/>
+  <axis xyz="1.0 0.0 0.0"/>
+  <limit upper="1.308997" lower="-1.745329" effort="100" velocity="100"/>
+</joint>
+<joint name="dummy_joint3" type="revolute">
+  <origin xyz="0.03565 0.0 0.168" rpy="0 0 0"/>
+  <parent link="link2_3_v4_1"/>
+  <child link="link4_v3_1"/>
+  <axis xyz="1.0 -0.0 0.0"/>
+  <limit upper="1.396263" lower="-1.570796" effort="100" velocity="100"/>
+</joint>
+<joint name="dummy_joint4" type="revolute">
+  <origin xyz="-0.013162 0.001043 0.062467" rpy="0 0 0"/>
+  <parent link="link4_v3_1"/>
+  <child link="link5_v3_1"/>
+  <axis xyz="-0.0 1.0 0.0"/>
+  <limit upper="3.141593" lower="-3.141593" effort="100" velocity="100"/>
+</joint>
+<joint name="dummy_joint5" type="revolute">
+  <origin xyz="0.0223 0.11 0.0" rpy="0 0 0"/>
+  <parent link="link5_v3_1"/>
+  <child link="link6_v3_1"/>
+  <axis xyz="1.0 0.0 0.0"/>
+  <limit upper="1.919862" lower="-1.745329" effort="100" velocity="100"/>
+</joint>
+<joint name="dummy_joint6" type="revolute">
+  <origin xyz="-0.021 0.117 0.0" rpy="0 0 0"/>
+  <parent link="link6_v3_1"/>
+  <child link="link7_v3_1"/>
+  <axis xyz="0.0 1.0 0.0"/>
+  <limit upper="1.919862" lower="-1.745329" effort="100" velocity="100"/>
+</joint>
  <!-- Piper 機器人連接
   <joint name="zyx_piper_base_joint" type="fixed">

File: src/piper_description/urdf/piper_description_d405_marco.xacro (robot description, xacro)
@@ -314,5 +314,5 @@
     <link name="${prefix}_gripper_point"/>
 <joint name="${prefix}_gripper_points" type="fixed">
-   <origin xyz="-0.0 0.0 0.11" rpy="-0.0 0.0 -0.0"/>
+   <origin xyz="-0.0 0.0 0.11" rpy="-0.0 0.0 -3.14"/>
     <parent link="${prefix}_link6"/>
     <child link="${prefix}_gripper_point"/>
