Commit message: updata_dual_transfer

File: src/Dual-arm-robot/scout_description/urdf/combined_robot_doublearm.xacro (robot description, xacro)
@@ -22,11 +22,12 @@
     parent_link="link3_1_v1_1"
     xyz="0.0 -0.20 0.05"
-    rpy="0 0 0"/>
+    rpy="3.14 0 0"/>
  <!-- 第1台相機：掛在 arm1link6 -->
+  <!-- x="-0.06092" y="0.00551" z="0.030946" roll="-0.29119" pitch="0.016918" yaw="-1.6641" 正手 -->
   <xacro:d405_camera
     prefix="cam1"
     parent_link="arm1_link6"
-    x="-0.06092" y="0.00551" z="0.030946"
-    roll="-0.29119" pitch="0.016918" yaw="-1.6641"
+    x="-0.06152" y="-0.00327" z="0.030479"
+    roll="0.29119" pitch="-0.020223" yaw="1.433"
     use_nominal_extrinsics="false"/>
   <!-- 在 link3_1_v1_1 右邊掛載第二支手臂  -->
@@ -35,5 +36,5 @@
     parent_link="link3_1_v1_1"
    xyz="0.0 0.20 0.05"
-    rpy="0 0 0"/>
+    rpy="3.14 0 0"/>
     <!-- 第2台相機：掛在 arm2link6 -->
     <!---->

File: src/Dual-arm-robot/scout_description/urdf/combined_robot_doublearm_nocar.xacro (robot description, xacro)
@@ -21,12 +21,17 @@
     prefix="arm1"
     parent_link="base_link"
-    xyz="0.0 -0.20 0.05"
-    rpy="0 0 0"/>
- <!-- 第1台相機：掛在 arm1link6 -->
+    xyz="0.0 -0.200 0.05"
+    rpy="3.14 0 0"/>
+    <!--rpy="0 0 0"/>-->
+ <!-- 第1台相機：掛在 arm1link6
+       正手
+     x="-0.06092" y="0.00551" z="0.030946"
+    roll="-0.29119" pitch="0.016918" yaw="1.4759"
+ -->
   <xacro:d405_camera
     prefix="cam1"
     parent_link="arm1_link6"
-    x="-0.06092" y="0.00551" z="0.030946"
-    roll="-0.29119" pitch="0.016918" yaw="-1.6641"
+     x="-0.10152" y="0.00327" z="0.030479"
+    roll="0.29119" pitch="-0.020223" yaw="1.433"
     use_nominal_extrinsics="false"/>
   <!-- 在 link3_1_v1_1 右邊掛載第二支手臂  -->
@@ -34,13 +39,18 @@
     prefix="arm2"
     parent_link="base_link"
-   xyz="0.0 0.20 0.05"
-    rpy="0 0 0"/>
+   xyz="0.0 0.200 0.05"
+   rpy="3.14 0 0"/>
+    <!--  rpy="0 0 0"/> -->
     <!-- 第2台相機：掛在 arm2link6 -->
-    <!---->
+    <!--
+       正手
+     x="-0.06092" y="0.00551" z="0.030946"
+    roll="-0.29119" pitch="0.016918" yaw="1.4759"
+    -->
   <xacro:d405_camera
     prefix="cam2"
     parent_link="arm2_link6"
-    x="-0.06092" y="0.00551" z="0.030946"
-    roll="-0.29119" pitch="0.016918" yaw="-1.6641"
+    x="-0.10152" y="0.00327" z="0.030479"
+    roll="0.29119" pitch="-0.020223" yaw="1.57"
     use_nominal_extrinsics="false"/>
  <!-- Piper 機器人連接

File: src/piper_description/urdf/piper_description_d405.xacro (robot description, xacro)
@@ -17,4 +17,11 @@
     <parent link="link6"/>
     <child link="d405_base_link"/>
+</joint>
+<link name="gripper_point"/>
+<joint name="gripper_points" type="fixed">
+      <!--<origin xyz="-0.064868 0.014226 0.029185" rpy="-0.283249 0.012335 -1.670768"/> -->
+   <origin xyz="-0.0 0.0 0.11" rpy="-0.0 0.0 -0.0"/>
+    <parent link="link6"/>
+    <child link="gripper_point"/>
 </joint>
 <!-- arm -->

File: src/piper_description/urdf/piper_description_d405_marco.xacro (robot description, xacro)
@@ -312,4 +312,10 @@
       <limit lower="-0.035" upper="0" effort="10" velocity="1" />
     </joint>
+    <link name="${prefix}_gripper_point"/>
+<joint name="${prefix}_gripper_points" type="fixed">
+   <origin xyz="-0.0 0.0 0.11" rpy="-0.0 0.0 -0.0"/>
+    <parent link="${prefix}_link6"/>
+    <child link="${prefix}_gripper_point"/>
+</joint>
   </xacro:macro>
 </robot>

Commit message: upate save 250925

File: src/Dual-arm-robot/scout_description/urdf/combined_robot_doublearm.xacro (robot description, xacro)
@@ -1,7 +1,7 @@
 <?xml version="1.0"?>
 <robot name="combined_robot" xmlns:xacro="http://www.ros.org/wiki/xacro">
-  <!-- 引入兩個機器人的Xacro文件
+  <!-- 引入兩個機器人的Xacro文件 -->
   <xacro:include filename="$(find scout_description)/urdf_zyx/zyx_R_1.xacro"/>
-  <xacro:include filename="$(find scout_description)/urdf/scout_v2.xacro"/>-->
+  <xacro:include filename="$(find scout_description)/urdf/scout_v2.xacro"/>
   <!-- <xacro:include filename="$(find piper_description)/urdf/piper_description.xacro"/>-->
     <!-- 引入 piper_arm_macro.xacro-->
@@ -54,22 +54,22 @@
     roll="0.29119" pitch="-0.020223" yaw="1.57"
     use_nominal_extrinsics="false"/>
- <!-- Piper 機器人連接
+ <!-- Piper 機器人連接 -->
   <joint name="zyx_piper_base_joint" type="fixed">
     <origin xyz="0.0 -0.5 0.0" rpy="1.57 1.57 0"/>
     <parent link="link3_1_v1_1"/>
     <child link="Piper_base_link"/>
-  </joint>-->
-  <!-- zyx_R_1 機器人連接
+  </joint>
+  <!-- zyx_R_1 機器人連接 -->
   <joint name="zyx_R_1_base_joint" type="fixed">
     <origin xyz="0.38 -0.14 0.19" rpy="0 0 0"/>
     <parent link="combined_base"/>
     <child link="zyx_R_1_base_link"/>
-  </joint>-->
-  <!-- scout_v2 機器人連接
+  </joint>
+  <!-- scout_v2 機器人連接 -->
   <joint name="scout_v2_base_joint" type="fixed">
     <origin xyz="0 0 0" rpy="0 0 0"/>
     <parent link="combined_base"/>
-    <child link="base_link"/>-->
-    <!--child link="scout_v2_base_link"/
-  </joint>-->
+    <child link="base_link"/>
+    <!--child link="scout_v2_base_link"/-->
+  </joint>
 </robot>

File: src/Dual-arm-robot/scout_description/urdf/combined_robot_triplearm_havecar.xacro (robot description, xacro)
@@ -2,16 +2,16 @@
 <robot name="combined_robot" xmlns:xacro="http://www.ros.org/wiki/xacro">
   <!-- 引入兩個機器人的Xacro文件
-  <xacro:include filename="$(find scout_description)/urdf_zyx/zyx_R_1.xacro"/>
-  <xacro:include filename="$(find scout_description)/urdf/scout_v2.xacro"/>-->
+  <xacro:include filename="$(find scout_description)/urdf_zyx/zyx_R_1.xacro"/>-->
+  <xacro:include filename="$(find scout_description)/urdf/scout_v2.xacro"/>
   <!-- <xacro:include filename="$(find piper_description)/urdf/piper_description.xacro"/>-->
     <!-- 引入 piper_arm_macro.xacro-->
-    <xacro:include filename="$(find Dual_piper_ROS2_description)/urdf/materials.xacro" />
-<xacro:include filename="$(find Dual_piper_ROS2_description)/urdf/Dual_piper_ROS2.trans" />
-<xacro:include filename="$(find Dual_piper_ROS2_description)/urdf/Dual_piper_ROS2.gazebo" />
-      <xacro:include filename="$(find realsense2_description)/urdf/_materials.urdf.xacro" />
-<xacro:include filename="$(find piper_description)/urdf/piper_description_d405_marco.xacro"/>
+  <xacro:include filename="$(find Dual_piper_ROS2_description)/urdf/materials.xacro" />
+  <xacro:include filename="$(find Dual_piper_ROS2_description)/urdf/Dual_piper_ROS2.trans" />
+  <xacro:include filename="$(find Dual_piper_ROS2_description)/urdf/Dual_piper_ROS2.gazebo" />
+  <xacro:include filename="$(find realsense2_description)/urdf/_materials.urdf.xacro" />
+  <xacro:include filename="$(find piper_description)/urdf/piper_description_d405_marco.xacro"/>
   <!-- 引入相機的Xacro文件 -->
-<xacro:include filename="$(find realsense_custom_description)/urdf/piper_double_d405_camera.urdf.xacro"/>
-<xacro:include filename="$(find realsense_custom_description)/urdf/piper_d435i_camera.urdf.xacro"/>
+  <xacro:include filename="$(find realsense_custom_description)/urdf/piper_double_d405_camera.urdf.xacro"/>
+  <xacro:include filename="$(find realsense_custom_description)/urdf/piper_d435i_camera.urdf.xacro"/>
   <!-- 定義統一的父連接點
   <link name="base_link">
@@ -22,5 +22,5 @@
   </link>
 -->
-<link name="base_link">
+<link name="combined_base">
   <inertial>
     <origin xyz="-0.0023454168511469727 -7.5124051764860745e-06 0.99353047899548718" rpy="0 0 0"/>
@@ -29,37 +29,32 @@
   </inertial>
   <visual>
-    <origin xyz="0 0 1.2" rpy="0 0 -1.57"/>
+    <!-- <origin xyz="0 0 1.2" rpy="0 0 -1.57"/> -->
+    <origin xyz="-0.5 -0.25 0.11" rpy="0 0 0"/>
     <geometry>
       <!-- <mesh filename="file://$(find Dual_piper_ROS2_description)/meshes/base_link.stl" scale="0.001 0.001 0.001"/> -->
-      <mesh filename="file://$(find dummy_piper_ROS2_description)/meshes/base_link.stl" scale="0.001 0.001 0.001"/>
-    </geometry>
-    <material name="silver"/>
-  </visual>
-  <collision>
-    <origin xyz="0 0 1.2" rpy="0 0 -1.57"/>
-    <geometry>
-      <mesh filename="file://$(find dummy_piper_ROS2_description)/meshes/base_link.stl" scale="0.001 0.001 0.001"/>
-    </geometry>
-  </collision>
-</link>
+      <mesh filename="file://$(find dummy_piper_ROS2_description)/meshes/body_asm.stl" scale="0.001 0.001 0.001"/>
+    </geometry>
+    <material name="silver"/>
+  </visual>
+  <collision>
+    <origin xyz="-0.5 -0.25 0.1" rpy="0 0 -1.57"/>
+    <geometry>
+      <mesh filename="file://$(find dummy_piper_ROS2_description)/meshes/body_asm.stl" scale="0.001 0.001 0.001"/>
+    </geometry>
+  </collision>
+</link>
+  <!-- <link name="combined_base">
+    <inertial>
+      <mass value="200"/>
+      <inertia ixx="20" iyy="20" izz="20" ixy="0" iyz="0" ixz="0"/>
+    </inertial>
+  </link> -->
 <!-- 在 link3_1_v1_1 左邊掛載第一支手臂
 <origin xyz="0.21 -0.0075 0.052" rpy="0 0 0"/>-->
   <xacro:piper_arm
     prefix="arm1"
-    parent_link="base_link"
-    xyz="0.0075 0.205 1.23"
+    parent_link="combined_base"
+    xyz="0.26 0.205 1.17"
     rpy="3.14 0 0"/>
-    <!--
-  <xacro:piper_arm
-    prefix="arm1"
-    parent_link="base_link"
-    xyz="0.0 -0.200 0.05"
-    rpy="3.14 0 0"/>-->
-    <!--rpy="0 0 0"/>-->
- <!-- 第1台相機：掛在 arm1link6
-       正手
-     x="-0.06092" y="0.00551" z="0.030946"
-    roll="-0.29119" pitch="0.016918" yaw="1.4759"
- -->
   <xacro:d405_camera
     prefix="cam1"
@@ -70,6 +65,6 @@
    <xacro:piper_arm
     prefix="arm2"
-    parent_link="base_link"
-   xyz="0.0075 -0.205 1.23"
+    parent_link="combined_base"
+   xyz="0.26 -0.205 1.17"
    rpy="3.14 0 0"/>
   <!-- 在 link3_1_v1_1 右邊掛載第二支手臂
@@ -90,6 +85,6 @@
     prefix="cam2"
     parent_link="arm2_link6"
-    x="-0.113152" y="-0.02" z="0.040479"
-    roll="0.0" pitch="-0.35" yaw="3.14"
+    x="-0.113152" y="-0.0" z="0.050479"
+    roll="0.35" pitch="0.0" yaw="1.57"
     use_nominal_extrinsics="false"/>
   <xacro:d435_camera
@@ -256,6 +251,6 @@
 </link>
 <joint name="Rigid77" type="fixed">
-  <origin xyz="-0.05 0.0 1.2708" rpy="0 0 -1.57"/>
-  <parent link="base_link"/>
+  <origin xyz="0.205 0.0 1.21" rpy="0 0 -1.57"/>
+  <parent link="combined_base"/>
   <child link="Gasket_v3_1"/>
 </joint>
@@ -319,9 +314,10 @@
     <child link="zyx_R_1_base_link"/>
   </joint>-->
-  <!-- scout_v2 機器人連接
+  <!-- scout_v2 機器人連接 -->
   <joint name="scout_v2_base_joint" type="fixed">
     <origin xyz="0 0 0" rpy="0 0 0"/>
     <parent link="combined_base"/>
-    <child link="base_link"/>-->
+    <child link="base_link"/>
+  </joint>
     <!--child link="scout_v2_base_link"/
   </joint>-->
