Commit message: total tidy

File: src/Dual-arm-robot/scout_description/urdf/combined_robot_triplearm_havecar.xacro (robot description, xacro)
@@ -67,5 +67,5 @@
     parent_link="combined_base"
    xyz="0.26 -0.205 1.17"
-   rpy="3.14 0 0"/>
+   rpy="3.14 0 0" />
   <!-- 在 link3_1_v1_1 右邊掛載第二支手臂
   <xacro:piper_arm
@@ -82,9 +82,15 @@
     roll="-0.29119" pitch="0.016918" yaw="1.4759"
     -->
-  <xacro:d405_camera
+  <!-- <xacro:d405_camera
     prefix="cam2"
     parent_link="arm2_link6"
     x="-0.113152" y="-0.0" z="0.050479"
     roll="0.35" pitch="0.0" yaw="1.57"
+    use_nominal_extrinsics="false"/> -->
+  <xacro:d405_camera
+    prefix="cam2"
+    parent_link="Gasket_v3_1"
+    x="0.0" y="0.106" z="-0.35"
+    roll="-1.57" pitch="0.0" yaw="0.0"
     use_nominal_extrinsics="false"/>
   <xacro:d435_camera
@@ -94,4 +100,16 @@
     roll="0.0" pitch="-0.0" yaw="1.57"
     use_nominal_extrinsics="false"/>
+<joint name="cam3_color_optical_joint" type="fixed">
+  <origin xyz="0 0 0" rpy="-1.5708 0 -1.5708"/>
+  <parent link="cam3_link"/>
+  <child link="cam3_color_optical_frame"/>
+</joint>
+<link name="cam3_color_optical_frame"/>
+<joint name="cam3_depth_optical_joint" type="fixed">
+  <origin xyz="0 0 0" rpy="-1.5708 0 -1.5708"/>
+  <parent link="cam3_link"/>
+  <child link="cam3_depth_optical_frame"/>
+</joint>
+<link name="cam3_depth_optical_frame"/>
 <link name="Gasket_v3_1">
   <inertial>
